Commit message: Some launch files fixes, new moveit2 config

File: src/models/ur5e_model_pkg/urdf/ur5e_camera.urdf.xacro (robot description, xacro)
@@ -72,5 +72,5 @@
   </joint>
   <joint name="gripper_joint" type="fixed">
-  <parent link="tool0"/>
+  <parent link="$(arg tf_prefix)tool0"/>
   <child link="gripper_base_link"/>
   <origin xyz="0 0 0" rpy="0 0 0"/>

File: src/ur5e_config_moveit/config/ur5e.ros2_control.xacro (robot description, xacro)
@@ -57,11 +57,4 @@
                 <state_interface name="velocity"/>
             </joint>
-            <joint name="right_finger_joint">
-                <command_interface name="position"/>
-                <state_interface name="position">
-                  <param name="initial_value">${initial_positions['right_finger_joint']}</param>
-                </state_interface>
-                <state_interface name="velocity"/>
-            </joint>
         </ros2_control>
     </xacro:macro>
